Commit message: [major] Add navigation stack with pure pursuit planner

File: urdf/macros.urdf.xacro (robot description, xacro)
@@ -5,5 +5,5 @@
     <origin xyz="0 0 0" rpy="0 0 0" />
     <geometry>
-      <mesh filename="package://auto_racecar/urdf/meshes/chassis.stl"/>
+      <mesh filename="package://auto_racecar/meshes/chassis.stl"/>
     </geometry>
   </xacro:macro>
@@ -17,5 +17,5 @@
     <origin xyz="0 0 0" rpy="-1.571 0 0" />
     <geometry>
-      <mesh filename="package://auto_racecar/urdf/meshes/wheel.stl"/>
+      <mesh filename="package://auto_racecar/meshes/wheel.stl"/>
     </geometry>
   </xacro:macro>
@@ -23,5 +23,5 @@
     <origin xyz="0 0 0" rpy="1.571 0 0" />
     <geometry>
-      <mesh filename="package://auto_racecar/urdf/meshes/wheel.stl"/>
+      <mesh filename="package://auto_racecar/meshes/wheel.stl"/>
     </geometry>
   </xacro:macro>
@@ -29,5 +29,5 @@
     <origin xyz="0 0 0" rpy="0 0 0" />
     <geometry>
-      <mesh filename="package://auto_racecar/urdf/meshes/imu.stl"/>
+      <mesh filename="package://auto_racecar/meshes/imu.stl"/>
     </geometry>
   </xacro:macro>
@@ -35,5 +35,5 @@
     <origin xyz="0.0134 0 0" rpy="0 0 0" />
     <geometry>
-      <mesh filename="package://auto_racecar/urdf/meshes/lidar.stl"/>
+      <mesh filename="package://auto_racecar/meshes/lidar.stl"/>
     </geometry>
   </xacro:macro>

File: urdf/racecar.urdf.xacro (robot description, xacro)
@@ -1,7 +1,7 @@
 <?xml version="1.0"?>
 <robot xmlns:xacro="http://www.ros.org/wiki/xacro" name="racecar">
-  <xacro:include filename="$(find auto_racecar)/urdf/urdf/macros.urdf.xacro"/>
-  <xacro:include filename="$(find auto_racecar)/urdf/urdf/materials.urdf.xacro"/>
-  <xacro:include filename="$(find auto_racecar)/urdf/urdf/racecar.gazebo"/>
+  <xacro:include filename="$(find auto_racecar)/urdf/macros.urdf.xacro"/>
+  <xacro:include filename="$(find auto_racecar)/urdf/materials.urdf.xacro"/>
+  <xacro:include filename="$(find auto_racecar)/urdf/racecar.gazebo"/>
   <!-- Base Link -->
   <link name="base_link"/>
